File: kicad/c65Keyb.kicad_pcb (KiCad board)
At the start: 2 copper layers, 93 x 160 mm, 94 parts, among them J2 JACK-PLUG1, Q1 8Mhz, SW1 TASTER, U1 STM32F407IET6__FI__, U2 744245, U3 744245, U4 744245, X3 M09?S-182, X4 MKDS_5_3-6,35, X5 M09?S-182

Commit message: Refill, check DRC
Parts:
- moved R38 0.67 mm to (134.3, 112.4)
Routing:
- net GND: track 130.6 -> 262.3 mm
- net Net-(R38-Pad2): track 15.0 -> 15.9 mm
Other:
- rule trace_min: 0 -> 0.0762
